Commit message: Update camera.xacro to move camera

File: kinova_description/urdf/camera.xacro (robot description, xacro)
@@ -16,5 +16,5 @@
         <parent link="m1n6s300_link_6"/>
         <child link="camera_link"/>
-        <origin xyz="0 0 0" rpy="0 1.5 0"/>
+        <origin xyz="0 0 -0.175" rpy="0 1.5 0"/>
     </joint>
     <link name="camera_link">
